File: TMC261-stepstick-v1.1.kicad_pcb (KiCad board)
At the start: 2 copper layers, 101 x 54.6 mm, 43 parts, among them P1 CONN_01X02, P2 CONN_02X03, P3 CONN_01X04, P4 CONN_01X04, P5 CONN_01X25, P6 CONN_01X04, P7 CONN_01X04, P8 CONN_01X04, U1 TMC261, U2 TMC261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

Commit message: ehm
Parts:
- removed G*** (x2): LOGO, graphics:Kiwi-silk
